File: FaceCam/Schematic/projects/FaceCam/FaceCam.sch (EAGLE design)
At the start: 17 parts, among them J1 AXE530127, J2 AXE530127, J3 AXE530127, J4 AXE530127, U1 LIF-MD6000-6MG81I, U2 CYUSB3064-BZXC, U3 TCA9548AMRGERVQFN-24

Commit message: Add regulators to library
Parts:
- added C1, C3, C5: 0.1uF, rcl:C-EUC0402
- added C2, C4: 2.2uF, rcl:C-EUC0402
- added L1, L2: BLM15HB121SN1, inductors:BLM15HB121SN1
- added U4: M25P40-VMN6TPB, library:M25P40-VMN6TPB
- added U5: TPS72012DRVR, TPS72012DRVR:TPS72012DRVR
- added U6: ADP323ACPZ-R7, ADP323ACPZ-R7:ADP323ACPZ-R7
Connections:
- new net CH4_DATA0_N: U2.D0M
- new net CH4_DATA0_P: U2.D0P
- new net CH4_DATA1_N: U2.D1M
- new net CH4_DATA1_P: U2.D1P
- new net CX3_SPI_MISO: U2.MISO, U4.Q
- new net CX3_SPI_MOSI: U2.MOSI, U4.D
- new net CX3_SPI_SCK: U2.SCK, U4.C
- new net CX3_SPI_SSN: U2.SSN, U4.!S
- new net N$3: C1.1, U4.VCC
- new net VCC: L1.1, L2.1, U2.VDD1, U2.VDD2, U2.VDD3, U2.VDD4, U2.VDD5, U2.VDD6, U2.VDD7, U2.VDD_MIPI
- new net VCCA_DPHY0: C4.1, C5.1, L2.2, U1.VCCA_DPHY0
- new net VCCPLL_DPHY0: C2.1, C3.1, L1.2, U1.VCCPLL_DPHY0
- net CH4_DCK_TX_N: now also U2.CM
- net CH4_DCK_TX_P: now also U2.CP
- net DGND: now also C1.2, C2.2, C3.2, C4.2, C5.2, U4.VSS
Other:
- note added: "LIF-MD6000"
- note added: "MIPI connectors"
- moved on the sheet: J1, J2, J3, J4, R1, R10, R2, R3, R4, R5, R6, R7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

Commit message: Add power section by Timothy
Parts:
- added C10, C11, C12, C36, C37, C38, C39, C40, C41, C49, C50, C6, C7, C8, C9: 1uF, rcl:C-EUC0402
- added C13, C15, C16, C17, C18, C19, C20, C21, C22, C23, C24, C28, C29, C30, C31, C32, C33, C34, C35, C42, C43, C47, C48: 0.1uF, rcl:C-EUC0402
- added C14: 2.2uF, rcl:C-EUC0402
- added C25, C26: 22uF, resistor:C-EUC0805
- added C27, C46: 4.7uF, rcl:C-EUC0402
- added C44: 4.7uF, resistor:C-EUC0805
- added C45: 0.047uF, rcl:C-EUC0402
- added D1: SMF5.0AT1, diode:SMF5.0AT1
- added D2, D3: PGB1010402KR, diode:PGB1010402KR
- added EMI4183: EMI4183, yhtomit_ICs:EMI4183
- added FB, FB1: 2.2A, Nordic_nRF:INDUCTOR_0402_N
- added JP1: (no value), pinhead:PINHD-2X5
- added JP2: (no value), pinhead:PINHD-1X10
- added L6: BLM15HG601SN1, inductors:BLM15HG601SN1
- added LED1: (no value), eagle-ltspice:LED_ESML0603
- added Q1, Q2: (no value), crystal-geyer_V1_0:KXO-PXO/XO-V94
- added R11, R12, R13: 4.7k, rcl:R-US_R0402
- added R14: 100k, rcl:R-US_R0402
- added R15, R18, R21: 200k, rcl:R-US_R0402
- added R16: 35.7k, rcl:R-US_R0402
- added R17, R20, R23: 1k, rcl:R-US_R0402
- added R19: 43.2k, rcl:R-US_R0402
- added R22: 76.8k, rcl:R-US_R0402
- added R24, R30, R31: 1M, rcl:R-US_R0402
- added R25, R26: 51, rcl:R-US_R0402
- added R27, R28: 10k, rcl:R-US_R0402
- added R29: 0, rcl:R-US_R0402
- added TP1, TP2, TP3: TPB1,27, testpad:TPB1,27
- added TS1: RCLAMP0524J.TCT, library:RCLAMP0524J.TCT
- added U$1, U$2: 100nH, 300ma, Nordic_nRF:INDUCTOR_0402_N
- added U7: TLV70215DBVR, library:TLV70215DBVR
- added U8: NCP361SNT1G, library:NCP361SNT1G
- added U9: TLV70225, library:TLV70225
- U6: value ADP323ACPZ-R7 -> ADP323ACPZ-R7_ADP323ACPZ-R7; device ADP323ACPZ-R7:ADP323ACPZ-R7 -> FaceCam:ADP323ACPZ-R7_ADP323ACPZ-R7
Connections:
- removed net VCC: L1.1, L2.1, U2.VDD1, U2.VDD2, U2.VDD3, U2.VDD4, U2.VDD5, U2.VDD6, U2.VDD7, U2.VDD_MIPI
- removed net VDD: J1.P5, J2.P5, J3.P5, J4.P5, R10.2, R3.2, R4.2, R5.2, R6.2, R7.2, R8.2, R9.2, U3.VCC
- new net +1V2: C14.2, C33.1, C34.1, C35.1, FB.1, FB1.1, JP1.1, L1.1, L2.1, U$1.1, U1.VCC1, U1.VCC2, U1.VCCGPLL, U2.VDD1, U2.VDD2, U2.VDD3, U2.VDD4, U2.VDD5, U2.VDD6, U2.VDD7, U2.VDD_MIPI, U5.OUT
- new net +1V5: C41.2, U7.OUT
- new net +1V8: C10.1, C15.1, C16.1, C17.1, C18.1, C29.1, C30.1, C31.1, C32.1, C39.2, C43.1, C48.1, J1.P5, J2.P5, J3.P5, J4.P5, Q1.VDD, Q2.VDD, R10.2, R21.1, R3.2, R4.2, R5.2, R6.2, R7.2, R8.2, R9.2, U$2.1, U1.VCCIO0, U1.VCCIO1, U1.VCCIO12, U1.VCCIO2, U1.VCCIO21, U2.VDDIO1_1, U2.VDDIO1_2, U2.VDDIO2, U3.VCC, U6.VOUT1
- new net +2V5: C50.2, R29.2, U9.OUT
- new net +2V8: C38.2, C9.1, R18.1, U6.VOUT2
- new net +3V3: C1.1, C11.1, C19.1, C36.2, R12.2, R13.2, R14.2, R15.1, U2.VDDIO3, U4.VCC, U6.VOUT3
- new net +5V: C12.2, C13.2, C22.1, C37.2, C40.2, C49.2, C6.2, C7.2, C8.2, U2.VUSB, U5.BIAS, U5.EN, U5.IN, U6.EN1, U6.EN2, U6.EN3, U6.VBIAS, U6.VIN1/VIN2, U6.VIN3, U7.EN, U7.IN, U8.OUT, U9.EN, U9.IN
- new net AVDD: C46.1, C47.1, U$1.2, U2.AVDD
- new net CH4_DCK_N: EMI4183.IN1-, U1.DPHY0_CKN
- new net CH4_DCK_P: EMI4183.IN1+, U1.DPHY0_CKP
- new net CY_RST: JP1.10, R28.1, U2.RESET
- new net CY_TCK: JP1.4, U2.TCK
- new net CY_TDI: JP1.8, U2.TDI
- new net CY_TDO: JP1.6, U2.TDO
- new net CY_TMS: JP1.2, U2.TMS
- new net CY_TRST: U2.TRST
- new net FLAG: LED1.C, R30.2, U8.!FLAG
- new net FLASH_HOLD: R12.1, U2.GPIO18, U4.!HOLD
- new net FLASH_W: R11.2, U2.GPIO17, U4.!W
- new net I2C_RST: U2.GPIO19, U3.RESET_N
- new net I2C_SCL: U2.I2C_SCL, U3.SCL
- new net I2C_SDA: U2.I2C_SDA, U3.SDA
- new net N$10: R26.2, U2.REFCLK
- new net N$11: R27.1, U2.MIPI_RESET
- new net N$12: C36.1, R17.1
- new net N$14: TP1.TP, U2.HSYNC_TEST
- new net N$16: TP2.TP, U2.VSYNC_TEST
- new net N$17: TP3.TP, U2.PCLK_TEST
- new net N$21: R18.2, R19.1, R20.2, U6.FB2
- new net N$22: C38.1, R20.1
- new net N$23: R29.1, U1.VCCAUX
- new net N$25: R21.2, R22.1, R23.2, U6.FB1
- new net N$26: C39.1, R23.1
- new net N$27: C21.1, U2.SSTX-
- new net N$28: C20.1, U2.SSTX+
- new net N$33: JP2.7, TS1.IN1
- new net N$34: JP2.6, TS1.IN2
- new net N$35: JP2.5, TS1.IN3
- new net N$36: JP2.4, TS1.IN4
- new net N$4: D1.C, JP2.10, L6.2
- new net N$5: Q1.OUT, R25.1
- new net N$6: LED1.A, R31.2
- new net N$7: Q2.OUT, R26.1
- new net N$8: C45.1, JP2.3, R24.1
- new net N$9: R25.2, U2.CLKIN
- new net USB2_DATA_M: D3.2, JP2.9, U2.D-
- new net USB2_DATA_P: D2.2, JP2.8, U2.D+
- new net USB_SSRX_M: TS1.NC4, U2.SSRX-
- new net USB_SSRX_P: TS1.NC3, U2.SSRX+
- new net USB_SSTX_M: C21.2, TS1.NC1
- new net USB_SSTX_P: C20.2, TS1.NC2
- new net VBUS: C42.1, C44.1, L6.1, R30.1, R31.1, U8.IN
- new net VCC1P2_FX3_RX: C23.1, C26.1, FB1.2, U2.U3RXVDDQ
- new net VCC1P2_FX3_TX: C24.1, C25.1, FB.2, U2.U3TXVDDQ
- new net VCCIO_CLK: C27.1, C28.1, R28.2, U$2.2, U2.CVDDQ
- net CH4_DATA0_N: now also EMI4183.IN2-, U1.DPHY0_DN0; no longer U2.D0M
- net CH4_DATA0_P: now also EMI4183.IN2+, U1.DPHY0_DP0; no longer U2.D0P
- net CH4_DATA0_TX_N: now also EMI4183.OUT2-, U2.D0M; no longer U1.DPHY0_DN0
- net CH4_DATA0_TX_P: now also EMI4183.OUT2+, U2.D0P; no longer U1.DPHY0_DP0
- net CH4_DATA1_N: now also EMI4183.IN3-, U1.DPHY0_DN1; no longer U2.D1M
- net CH4_DATA1_P: now also EMI4183.IN3+, U1.DPHY0_DP1; no longer U2.D1P
- net CH4_DATA1_TX_N: now also EMI4183.OUT3-, U2.D1M; no longer U1.DPHY0_DN1
- net CH4_DATA1_TX_P: now also EMI4183.OUT3+, U2.D1P; no longer U1.DPHY0_DP1
- net CH4_DCK_TX_N: now also EMI4183.OUT1-; no longer U1.DPHY0_CKN
- net CH4_DCK_TX_P: now also EMI4183.OUT1+; no longer U1.DPHY0_CKP
- net CX3_SPI_SCK: now also R14.1
- net CX3_SPI_SSN: now also R13.1
- net DGND: now also C10.2, C11.2, C12.1, C13.1, C14.1, C15.2, C16.2, C17.2, C18.2, C19.2, C22.2, C23.2, C24.2, C25.2, C26.2, C27.2, C28.2, C29.2, C30.2, C31.2, C32.2, C33.2, C34.2, C35.2, C37.1, C40.1, C41.1, C42.2, C43.2, C44.2, C45.2, C46.2, C47.2, C48.2, C49.1, C50.1, C6.1, C7.1, C8.1, C9.2, D1.A, D2.1, D3.1, EMI4183.GND@1, EMI4183.GND@2, EMI4183.GND@3, EMI4183.GND@4, JP1.3, JP1.5, JP1.9, JP2.1, JP2.2, Q1.GND, Q2.GND, R11.1, R16.2, R19.2, R22.2, R24.2, R27.2, TS1.GND1, TS1.GND2, U1.GNDA1_DPHY1, U1.GNDA_DPHY0, U1.GNDGPLL, U1.GNDPLL_DPHYX, U2.AVSS, U2.U3VSSQ, U5.EP, U5.GND, U6.EP, U6.GND, U7.GND, U8.!EN, U8.GND, U9.GND
- net N$3: now also R15.2, R16.1, R17.2, U6.FB3; no longer C1.1, U4.VCC
Other:
- note added: "Flag connected to or LED to indicate when there is overvoltage (optional)"
- note added: "MIPI to USB bridge"
- note added: "NCP361 disconnects systems at its output when the input voltage exceeds the overvoltage threshold (5.675 V)"
- note added: "Notes: - FB - Ferrite Beads"
- note added: "Place C20 and C21 next to CX3 IC"
- note added: "Protection against ESD"
- note added: "USB and Power Supply"
- note added: "Used to reduce effects of ESD in MIPI lanes"
- note added: "we will need to place an USB 3.0 connector instead of the pin header"
- moved on the sheet: C1, R1, U2, U4, U5, U6

Commit message: Preliminary schematic
Parts:
- added D4: GREEN, SparkFun-LED:LED-GREEN0603
- added JP3: (no value), pinhead:PINHD-1X3
- added R32, R33: 1k, rcl:R-US_R0402
- added R34, R35, R36: 10k, rcl:R-US_R0402
- added R37, R38, R42: 0, rcl:R-US_R0402
- added R39, R40, R41, R43: DNP, rcl:R-US_R0402
- added R44: 680R, rcl:R-US_R0402
Connections:
- new net CAM_SEL: R39.2, R42.2, U1.PB47
- new net CDONE: D4.A, R41.2, R44.1, U1.PB49
- new net CRESET_B: U1.CRESET_B, U2.GPIO20
- new net CX3_PMODE0: R34.1, U2.GPIO30
- new net CX3_PMODE1: R35.1, U2.GPIO31
- new net CX3_PMODE2: R36.2, U2.GPIO32
- new net CX3_UART_RX: JP3.2, U2.RX
- new net CX3_UART_TX: JP3.1, U2.TX
- new net GPIO21: U2.GPIO21
- new net GPIO22: R42.1, U2.GPIO22
- new net GPIO23: R43.1, U2.GPIO23
- new net GPIO_21: R41.1
- new net MIPI_CAM_RESET: R37.1, R40.2, R43.2, U1.PB48
- new net N$13: R37.2, U2.XRST
- new net N$15: R38.2, U2.XSHUTDOWN
- new net XSHUTDOWN: J1.P8, J2.P8, J3.P8, J4.P8, R38.1
- net +1V8: now also J1.P9, J2.P9, J3.P9, J4.P9, R32.2, R33.2, R34.2, R35.2, R44.2
- net DGND: now also JP3.3, R36.1
- net I2C_SCL: now also R32.1, R40.1, U1.PB52
- net I2C_SDA: now also R33.1, R39.1, U1.PB53
Other:
- moved on the sheet: C18, C29, C30, C31, C32, C33, C34, C35, C48, Q1, Q2, R1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
